Commit message: refactored env code for modular rooms and fixed unhandled preprocessors

File: softlearning/environments/gym/locobot/urdf/locobot_description.urdf (robot description, URDF)
Before this commit: robot locobot, 25 links, 24 joints
Links:
- link base_link: geometry collision cylinder length=0.120 radius=0.178; visual mesh filename=meshes/main_body.dae

Commit message: imported new locobot model

File: softlearning/environments/gym/locobot/urdf/locobot_description.urdf (robot description, URDF)
Before this commit: robot locobot, 25 links, 24 joints
Links:
- added link battery_link, mass 1.194; collision mesh filename=meshes/battery.stl scale=0.001 0.001 0.001; visual mesh filename=meshes/battery.stl scale=0.001 0.001 0.001
- link ar_tag: mass 0.00202622634619862 -> 0.0202622634619862
- link arm_base_link: mass 0.0531491686912019 -> 0.379673; geometry collision mesh filename=meshes/mobile_base.stl scale=0.001 0.001 0.001; visual mesh filename=meshes/mobile_base.stl scale=0.001 0.001 0.001
- link base_link: geometry collision cylinder length=0.10938 radius=0.178; visual mesh filename=meshes/main_body.dae
- link cam_mount: mass 0.0508068698311304 -> 2.091937; geometry collision mesh filename=meshes/cam_mount.stl scale=0.001 0.001 0.001; visual mesh filename=meshes/cam_mount.stl scale=0.001 0.001 0.001
- link camera_link: mass 0.00381925651163644 -> 0.0381925651163644
- link elbow_link: mass 0.0212482745791037 -> 0.212482745791037
- link finger_l: mass 0.00121931459003603 -> 0.0121931459003603
- link finger_r: mass 0.00121931459003602 -> 0.0121931459003602
- link forearm_link: mass 0.018746427435805 -> 0.18746427435805
- link gripper_link: mass 0.00795745052466434 -> 0.0795745052466434
- link head_pan_link: mass 0.00182769203076134 -> 0.0182769203076134
- link head_tilt_link: mass 0.00547677687275323 -> 0.0547677687275323
- link plate_1: mass 0.0640128902693298 -> 0.27854; geometry collision mesh filename=meshes/plate_bottom.stl scale=0.001 0.001 0.001; visual mesh filename=meshes/plate_bottom.stl scale=0.001 0.001 0.001
- link plate_2: mass 0.0640128902693298 -> 0.27854; geometry collision mesh filename=meshes/plate_top.stl scale=0.001 0.001 0.001; visual mesh filename=meshes/plate_top.stl scale=0.001 0.001 0.001
- link shoulder_link: mass 0.0119861197293521 -> 0.119861197293521
- link wrist_link: mass 0.00605921736680362 -> 0.0605921736680362
Joints:
- added joint battery_link_joint: type fixed, parent plate_2, child battery_link, origin xyz=-0.09703321 0 0.005375 rpy=0 0 0, axis 0 0 0
- joint arm_base_link_joint: origin xyz=0 0 0.001 rpy=0 0 0 -> xyz=0 0 0.002375 rpy=0 0 0
- joint cam_mount_joint: origin xyz=-0.03751 0 0.1331 rpy=0 0 0 -> xyz=-0.03751 0 0.13775 rpy=0 0 0
- joint head_pan_joint: origin xyz=0.0240154841629213 -0.000373468229198185 0.4065 rpy=0 0 0 -> xyz=0.01755 -0.00008 0.3975 rpy=0 0 0
- joint joint_1: origin xyz=0 0 0.072 rpy=0 0 0 -> xyz=0 0 0.0655 rpy=0 0 0
- joint plate_2_joint: origin xyz=0 0 0.0047625 rpy=0 0 0 -> xyz=0 0 0.00475 rpy=0 0 0

Commit message: added new locobot model and offset camera

File: softlearning/environments/gym/locobot/urdf/locobot_description.urdf (robot description, URDF)
Before this commit: robot locobot, 26 links, 25 joints
Joints:
- joint cam_mount_joint: origin xyz=-0.03751 0 0.13775 rpy=0 0 0 -> xyz=-0.03751 0.0 0.13775 rpy=0 0 0
- joint head_pan_joint: origin xyz=0.01755 -0.00008 0.3975 rpy=0 0 0 -> xyz=0.01755 -0.10000 0.3975 rpy=0 0 0

Commit message: train autoregressive grasping

File: softlearning/environments/gym/locobot/urdf/locobot_description.urdf (robot description, URDF)
Before this commit: robot locobot, 26 links, 25 joints
Links:
- added link camera_lens_link, mass 0.000001; visual box size=0.02 0.02 0.02
Joints:
- added joint camera_lens_link: type fixed, parent camera_link, child camera_lens_link, origin xyz=0.02 0 0 rpy=0 0 0, axis 0 0 0
- joint head_pan_joint: origin xyz=0.01755 -0.10000 0.3975 rpy=0 0 0 -> xyz=0.01755 -0.00000 0.3975 rpy=0 0 0

Commit message: shift camera

File: softlearning/environments/gym/locobot/urdf/locobot_description.urdf (robot description, URDF)
Before this commit: robot locobot, 27 links, 26 joints
Links:
- link camera_lens_link: geometry visual box size=0.002 0.002 0.002
Joints:
- joint head_pan_joint: origin xyz=0.01755 -0.00000 0.3975 rpy=0 0 0 -> xyz=0.01755 -0.10000 0.3975 rpy=0 0 0

Commit message: New version of the env

File: softlearning/environments/gym/locobot/urdf/locobot_description.urdf (robot description, URDF)
Before this commit: robot locobot, 27 links, 26 joints
Joints:
- joint head_pan_joint: origin xyz=0.01755 -0.00000 0.3975 rpy=0 0 0 -> xyz=0.11755 -0.10000 0.3975 rpy=0 0 0

Commit message: added multistep grasping env

File: softlearning/environments/gym/locobot/urdf/locobot_description.urdf (robot description, URDF)
Before this commit: robot locobot, 27 links, 26 joints
Links:
- added link aux_camera_lens_link, mass 0.000001; visual box size=0.002 0.002 0.002
Joints:
- removed joint camera_lens_link
- added joint aux_camera_lens_joint: type fixed, parent camera_link, child aux_camera_lens_link, origin xyz=0.02 0.1 0 rpy=0 0 0, axis 0 0 0
- added joint camera_lens_joint: type fixed, parent camera_link, child camera_lens_link, origin xyz=0.02 -0.1 0 rpy=0 0 0, axis 0 0 0
- joint head_pan_joint: origin xyz=0.01755 -0.10000 0.3975 rpy=0 0 0 -> xyz=0.01755 -0.00000 0.3975 rpy=0 0 0
