Commit message: separated dual cam and single cam

File: softlearning/environments/gym/locobot/urdf/locobot_description_dual_cam.urdf (robot description, URDF)
Before this commit: robot locobot, 28 links, 27 joints
Joints:
- joint aux_camera_lens_joint: origin xyz=0.02 0 0 rpy=0 0 0 -> xyz=0.02 0.1 0 rpy=0 0 0
- joint camera_lens_joint: origin xyz=0.02 0 0 rpy=0 0 0 -> xyz=0.02 -0.1 0 rpy=0 0 0
